Commit message: Initial migration to ROS 2; largely untested, probably a few bugs to work through. But the basic models load in rviz and the packages build, so that's a start.

File: lego_spike_description/urdf/lego_dimensions.urdf.xacro (robot description, xacro)
@@ -1,5 +1,4 @@
 <?xml version="1.0" ?>
 <robot xmlns:xacro="http://wiki.ros.org/xacro">
-  <xacro:property name="pi" value="3.141592653589793"/>
   <!--
     Lego nominal dimensions.  These are useful for applying XYZ offsets between components so
